Commit message: rplidar

File: urdf/sensors/rplidar_a2.urdf.xacro (robot description, xacro)
@@ -9,29 +9,29 @@
 	</xacro:macro>
 	<xacro:macro name="sensor_rplidar" params="parent">
-    <joint name="laser" type="fixed">
-		  <origin xyz="0 0 0.42" rpy="0 0 0" />
-			<parent link="${parent}" />
-			<child link="base_laser_link" />
-	  </joint>
-		<link name="base_laser_link">
-			<visual>
-				<origin xyz="0 0 0" rpy="0 0 0"/>
-				<xacro:lidar_geometry />
-				<material name="blue">
-					<color rgba="0 0 .8 1"/>
-				</material>
-			</visual>
-			<collision>
-				<origin xyz="0 0 0" rpy="0 0 0"/>
-				<xacro:lidar_geometry />
-		  </collision>
-		  <inertial>
-				<mass value="0.19" />
-				<origin xyz="0 0 0" />
-				<inertia ixx="0.003881243" ixy="0.0" ixz="0.0"
-				         iyy="0.000498940" iyz="0.0"
-				         izz="0.003879257" />
-		  </inertial>
-		</link>
+    	<joint name="laser" type="fixed">
+		<origin xyz="0 0 0.42" rpy="0 0 0" />
+		<parent link="${parent}" />
+		<child link="base_laser_link" />
+	</joint>
+	<link name="base_laser_link">
+		<visual>
+			<origin xyz="0 0 0" rpy="0 0 0"/>
+			<xacro:lidar_geometry />
+			<material name="blue">
+				<color rgba="0 0 .8 1"/>
+			</material>
+		</visual>
+		<collision>
+			<origin xyz="0 0 0" rpy="0 0 0"/>
+			<xacro:lidar_geometry />
+		</collision>
+		<inertial>
+			<mass value="0.19" />
+			<origin xyz="0 0 0" />
+			<inertia ixx="0.003881243" ixy="0.0" ixz="0.0"
+				 iyy="0.000498940" iyz="0.0"
+				 izz="0.003879257" />
+		</inertial>
+	</link>
 	</xacro:macro>
 </robot>
